File: bmp-c.kicad_pcb (KiCad board)
At the start: 2 copper layers, 37.5 x 16.5 mm, 60 parts, among them J1 TYPE-C-31-M-12, J3 FTSH-107-01-F-DV-K, Q1 DMG1023UV, Q2 DMG1024UV, SW1 B3U-1000P, U1 USBLC6-2P6, U2 74LVC2T45GT, U3 74LVC2T45GT, U4 74LVC2T45GT, U5 74LVC2T45GT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

Commit message: Fix up known issues.
Parts:
- D2: value LED GREEN -> LED BLUE
- D3: value LED ORANGE -> LED GREEN
- FB1: value Ferrite_Bead_Small -> 330R @ 100MHz
- moved LOGO1 0.30 mm to (92.0, 80.2)
